File: keeb/keeb.kicad_pcb (KiCad board)
At the start: 2 copper layers, 100 parts, among them SW1 Switch, SW10 Switch, SW11 Switch, SW12 Switch, SW13 Switch, SW14 Switch, SW15 Switch, SW16 Switch, SW17 Switch, SW18 Switch, SW19 Switch, SW2 Switch, SW20 Switch, SW21 Switch, SW22 Switch, SW23 Switch, SW24 Switch, SW25 Switch, SW26 Switch, SW27 Switch, SW28 Switch, SW29 Switch, SW3 Switch, SW30 Switch, SW31 Switch, SW32 Switch, SW33 Switch, SW34 Switch, SW35 Switch, SW36 Switch, SW37 Switch, SW38 Switch, SW39 Switch, SW4 Switch, SW40 Switch, SW41 Switch, SW42 Switch, SW43 Switch, SW44 Switch, SW45 Switch, SW46 Switch, SW47 Switch, SW48 Switch, SW5 Switch, SW6 Switch, SW7 Switch, SW8 Switch, SW9 Switch, U1 RP2040_Zero, U2 RP2040_Zero, U3 TRRS, U4 TRRS

Commit message: things
Parts:
- removed D1, D10, D11, D12, D13, D14, D15, D16, D17, D18, D19, D2, D20, D21, D22, D23, D24, D25, D26, D27, D28, D29, D3, D30, D31, D32, D33, D34, D35, D36, D37, D38, D39, D4, D40, D41, D42, D43, D44, D45, D46, D47, D48, D5, D6, D7, D8, D9: 1N4148WT, Diode_SMD:D_SOD-523
- removed SW1, SW10, SW11, SW12, SW13, SW14, SW15, SW16, SW17, SW18, SW19, SW2, SW20, SW21, SW22, SW23, SW24, SW25, SW26, SW27, SW28, SW29, SW3, SW30, SW31, SW32, SW33, SW34, SW35, SW36, SW37, SW38, SW39, SW4, SW40, SW41, SW42, SW43, SW44, SW45, SW46, SW47, SW48, SW5, SW6, SW7, SW8, SW9: Switch, ScottoKeebs_MX:MX_PCB_1.00u
- removed U1, U2: RP2040_Zero, ScottoKeebs_MCU:RP2040_Zero
- removed U3, U4: TRRS, ScottoKeebs_Components:TRRS_PJ-320A
- added LController1: ~, ScottoKeebs_MCU:Adafruit_KB2040, F.Cu at (157.0, -104.0)
- added LeftD1: Diode, Diode_THT:D_DO-35_SOD27_P7.62mm_Horizontal, F.Cu at (44.7, -38.9)
- added LeftD10: Diode, Diode_THT:D_DO-35_SOD27_P7.62mm_Horizontal, F.Cu at (44.7, -62.3)
- added LeftD11: Diode, Diode_THT:D_DO-35_SOD27_P7.62mm_Horizontal, F.Cu at (44.7, -76.3)
- added LeftD12: Diode, Diode_THT:D_DO-35_SOD27_P7.62mm_Horizontal, F.Cu at (44.7, -99.7)
- added LeftD13: Diode, Diode_THT:D_DO-35_SOD27_P7.62mm_Horizontal, F.Cu at (44.7, -24.8)
- added LeftD14: Diode, Diode_THT:D_DO-35_SOD27_P7.62mm_Horizontal, F.Cu at (44.7, -52.9)
- added LeftD15: Diode, Diode_THT:D_DO-35_SOD27_P7.62mm_Horizontal, F.Cu at (44.7, -81.0)
- added LeftD16: Diode, Diode_THT:D_DO-35_SOD27_P7.62mm_Horizontal, F.Cu at (44.7, -104.4)
- added LeftD17: Diode, Diode_THT:D_DO-35_SOD27_P7.62mm_Horizontal, F.Cu at (44.7, -43.5)
- added LeftD18: Diode, Diode_THT:D_DO-35_SOD27_P7.62mm_Horizontal, F.Cu at (44.7, -66.9)
- added LeftD19: Diode, Diode_THT:D_DO-35_SOD27_P7.62mm_Horizontal, F.Cu at (44.7, -90.3)
- added LeftD2: Diode, Diode_THT:D_DO-35_SOD27_P7.62mm_Horizontal, F.Cu at (44.7, -48.2)
- added LeftD3: Diode, Diode_THT:D_DO-35_SOD27_P7.62mm_Horizontal, F.Cu at (44.7, -71.6)
- added LeftD4: Diode, Diode_THT:D_DO-35_SOD27_P7.62mm_Horizontal, F.Cu at (44.7, -95.0)
- added LeftD5: Diode, Diode_THT:D_DO-35_SOD27_P7.62mm_Horizontal, F.Cu at (44.7, -29.5)
- added LeftD6: Diode, Diode_THT:D_DO-35_SOD27_P7.62mm_Horizontal, F.Cu at (44.7, -57.6)
- added LeftD7: Diode, Diode_THT:D_DO-35_SOD27_P7.62mm_Horizontal, F.Cu at (44.7, -85.7)
- added LeftD8: Diode, Diode_THT:D_DO-35_SOD27_P7.62mm_Horizontal, F.Cu at (44.7, -109.1)
- added LeftD9: Diode, Diode_THT:D_DO-35_SOD27_P7.62mm_Horizontal, F.Cu at (44.7, -34.2)
- added LeftSW1: Switch, ScottoKeebs_MX:MX_PCB_1.00u, F.Cu at (77.5, -93.0)
- added LeftSW10: Switch, ScottoKeebs_MX:MX_PCB_1.00u, F.Cu at (115.5, -87.5)
- added LeftSW11: Switch, ScottoKeebs_MX:MX_PCB_1.00u, F.Cu at (115.5, -68.5)
- added LeftSW12: Switch, ScottoKeebs_MX:MX_PCB_1.00u, F.Cu at (115.5, -49.4)
- added LeftSW13: Switch, ScottoKeebs_MX:MX_PCB_1.00u, F.Cu at (135.0, -100.5)
- added LeftSW14: Switch, ScottoKeebs_MX:MX_PCB_1.00u, F.Cu at (135.0, -81.5)
- added LeftSW15: Switch, ScottoKeebs_MX:MX_PCB_1.00u, F.Cu at (135.0, -62.5)
- added LeftSW16: Switch, ScottoKeebs_MX:MX_PCB_1.00u, F.Cu at (135.0, -43.4)
- added LeftSW17: Switch, ScottoKeebs_MX:MX_PCB_1.00u, F.Cu at (154.0, -73.0)
- added LeftSW18: Switch, ScottoKeebs_MX:MX_PCB_1.00u, F.Cu at (154.0, -54.0)
- added LeftSW19: Switch, ScottoKeebs_MX:MX_PCB_1.00u, F.Cu at (154.0, -35.0)
- added LeftSW2: Switch, ScottoKeebs_MX:MX_PCB_1.00u, F.Cu at (77.5, -74.0)
- added LeftSW3: Switch, ScottoKeebs_MX:MX_PCB_1.00u, F.Cu at (77.5, -55.0)
- added LeftSW4: Switch, ScottoKeebs_MX:MX_PCB_1.00u, F.Cu at (77.5, -36.0)
- added LeftSW5: Switch, ScottoKeebs_MX:MX_PCB_1.00u, F.Cu at (96.5, -97.5)
- added LeftSW6: Switch, ScottoKeebs_MX:MX_PCB_1.00u, F.Cu at (96.5, -78.5)
- added LeftSW7: Switch, ScottoKeebs_MX:MX_PCB_1.00u, F.Cu at (96.5, -59.5)
- added LeftSW8: Switch, ScottoKeebs_MX:MX_PCB_1.00u, F.Cu at (96.5, -40.5)
- added LeftSW9: Switch, ScottoKeebs_MX:MX_PCB_1.00u, F.Cu at (115.5, -106.5)
- added RController1: ~, ScottoKeebs_MCU:Adafruit_KB2040, F.Cu at (194.3, -104.0)
- added RightD1: Diode, Diode_THT:D_DO-35_SOD27_P7.62mm_Horizontal, F.Cu at (299.6, -25.7)
- added RightD10: Diode, Diode_THT:D_DO-35_SOD27_P7.62mm_Horizontal, F.Cu at (299.6, -48.7)
- added RightD11: Diode, Diode_THT:D_DO-35_SOD27_P7.62mm_Horizontal, F.Cu at (299.6, -76.4)
- added RightD12: Diode, Diode_THT:D_DO-35_SOD27_P7.62mm_Horizontal, F.Cu at (299.6, -108.7)
- added RightD13: Diode, Diode_THT:D_DO-35_SOD27_P7.62mm_Horizontal, F.Cu at (299.6, -44.1)
- added RightD14: Diode, Diode_THT:D_DO-35_SOD27_P7.62mm_Horizontal, F.Cu at (299.6, -53.4)
- added RightD15: Diode, Diode_THT:D_DO-35_SOD27_P7.62mm_Horizontal, F.Cu at (299.6, -81.0)
- added RightD16: Diode, Diode_THT:D_DO-35_SOD27_P7.62mm_Horizontal, F.Cu at (299.6, -99.5)
- added RightD17: Diode, Diode_THT:D_DO-35_SOD27_P7.62mm_Horizontal, F.Cu at (299.6, -34.9)
- added RightD18: Diode, Diode_THT:D_DO-35_SOD27_P7.62mm_Horizontal, F.Cu at (299.6, -62.6)
- added RightD19: Diode, Diode_THT:D_DO-35_SOD27_P7.62mm_Horizontal, F.Cu at (299.6, -90.2)
- added RightD2: Diode, Diode_THT:D_DO-35_SOD27_P7.62mm_Horizontal, F.Cu at (299.6, -67.2)
- added RightD3: Diode, Diode_THT:D_DO-35_SOD27_P7.62mm_Horizontal, F.Cu at (299.6, -71.8)
- added RightD4: Diode, Diode_THT:D_DO-35_SOD27_P7.62mm_Horizontal, F.Cu at (299.6, -104.1)
- added RightD5: Diode, Diode_THT:D_DO-35_SOD27_P7.62mm_Horizontal, F.Cu at (299.6, -39.5)
- added RightD6: Diode, Diode_THT:D_DO-35_SOD27_P7.62mm_Horizontal, F.Cu at (299.6, -58.0)
- added RightD7: Diode, Diode_THT:D_DO-35_SOD27_P7.62mm_Horizontal, F.Cu at (299.6, -85.6)
- added RightD8: Diode, Diode_THT:D_DO-35_SOD27_P7.62mm_Horizontal, F.Cu at (299.6, -94.9)
- added RightD9: Diode, Diode_THT:D_DO-35_SOD27_P7.62mm_Horizontal, F.Cu at (299.6, -30.3)
- added RightSW1: Switch, ScottoKeebs_MX:MX_PCB_1.00u, F.Cu at (200.3, -72.5)
- added RightSW10: Switch, ScottoKeebs_MX:MX_PCB_1.00u, F.Cu at (238.3, -70.0)
- added RightSW11: Switch, ScottoKeebs_MX:MX_PCB_1.00u, F.Cu at (238.3, -50.5)
- added RightSW12: Switch, ScottoKeebs_MX:MX_PCB_1.00u, F.Cu at (258.8, -63.1)
- added RightSW13: Switch, ScottoKeebs_MX:MX_PCB_1.00u, F.Cu at (258.8, -44.0)
- added RightSW14: Switch, ScottoKeebs_MX:MX_PCB_1.00u, F.Cu at (258.8, -101.0)
- added RightSW15: Switch, ScottoKeebs_MX:MX_PCB_1.00u, F.Cu at (258.8, -82.0)
- added RightSW16: Switch, ScottoKeebs_MX:MX_PCB_1.00u, F.Cu at (277.8, -92.0)
- added RightSW17: Switch, ScottoKeebs_MX:MX_PCB_1.00u, F.Cu at (277.8, -73.0)
- added RightSW18: Switch, ScottoKeebs_MX:MX_PCB_1.00u, F.Cu at (277.8, -54.0)
- added RightSW19: Switch, ScottoKeebs_MX:MX_PCB_1.00u, F.Cu at (277.8, -34.9)
- added RightSW2: Switch, ScottoKeebs_MX:MX_PCB_1.00u, F.Cu at (200.3, -53.5)
- added RightSW3: Switch, ScottoKeebs_MX:MX_PCB_1.00u, F.Cu at (200.3, -34.5)
- added RightSW4: Switch, ScottoKeebs_MX:MX_PCB_1.00u, F.Cu at (219.2, -62.4)
- added RightSW5: Switch, ScottoKeebs_MX:MX_PCB_1.00u, F.Cu at (219.2, -43.5)
- added RightSW6: Switch, ScottoKeebs_MX:MX_PCB_1.00u, F.Cu at (219.3, -100.9)
- added RightSW7: Switch, ScottoKeebs_MX:MX_PCB_1.00u, F.Cu at (219.3, -81.8)
- added RightSW8: Switch, ScottoKeebs_MX:MX_PCB_1.00u, F.Cu at (238.3, -108.0)
- added RightSW9: Switch, ScottoKeebs_MX:MX_PCB_1.00u, F.Cu at (238.3, -89.0)
Routing:
- net RightCol2: track 0.00 -> 479.1 mm
- net RightCol1: track 0.00 -> 327.4 mm
- net Net-(LeftD5-A): track 0.00 -> 270.0 mm
- net Net-(LeftD9-A): track 0.00 -> 255.3 mm
- net LeftRow2: track 0.00 -> 249.8 mm
- net RightRow3: track 0.00 -> 223.0 mm
- net Net-(LeftD13-A): track 0.00 -> 211.3 mm
- net RightRow2: track 0.00 -> 209.8 mm
- net LeftCol1: track 0.00 -> 209.3 mm, vias 0 -> 1
- net Net-(RightD2-A): track 0.00 -> 206.9 mm
- net LeftRow1: track 0.00 -> 187.5 mm
- net RightCol3: track 0.00 -> 184.1 mm, vias 0 -> 1
- net Net-(LeftD14-A): track 0.00 -> 179.0 mm
- net Net-(RightD12-A): track 0.00 -> 168.7 mm
- net RightRow4: track 0.00 -> 167.6 mm
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Other:
- board outline added: 270.3 x 100.6 mm
