File: keeb/keeb.kicad_sch (KiCad schematic)
At the start: 0 parts

Commit message: setup schem
Parts:
- added D1, D10, D11, D12, D13, D14, D15, D16, D17, D18, D19, D2, D20, D21, D22, D23, D24, D25, D26, D27, D28, D29, D3, D30, D31, D32, D33, D34, D35, D36, D37, D38, D39, D4, D40, D41, D42, D43, D44, D45, D46, D47, D48, D5, D6, D7, D8, D9: 1N4148WT, Diode_SMD:D_SOD-523, symbol Diode:1N4148WT
- added SW1, SW10, SW11, SW12, SW13, SW14, SW15, SW16, SW17, SW18, SW19, SW2, SW20, SW21, SW22, SW23, SW24, SW25, SW26, SW27, SW28, SW29, SW3, SW30, SW31, SW32, SW33, SW34, SW35, SW36, SW37, SW38, SW39, SW4, SW40, SW41, SW42, SW43, SW44, SW45, SW46, SW47, SW48, SW5, SW6, SW7, SW8, SW9: Switch, ScottoKeebs_MX:MX_PCB_1.00u, symbol ScottoKeebs:Placeholder_Switch
- added U1, U2: RP2040_Zero, ScottoKeebs_MCU:RP2040_Zero, symbol ScottoKeebs:MCU_RP2040_Zero
- added U3, U4: TRRS, ScottoKeebs_Components:TRRS_PJ-320A, symbol ScottoKeebs:Placeholder_TRRS
Connections:
- new net: D25.2 (A), SW25.2
- new net: D4.2 (A), SW4.2
- new net: D27.2 (A), SW27.2
- new net: D21.2 (A), SW21.2
- new net: D34.2 (A), SW34.2
- new net: U2.17 (26), U4.3 (RING1)
- new net: U2.18 (27), U4.2 (TIP)
- new net: U2.22 (GND), U4.1 (SLEEVE)
- new net: U2.23 (5V), U4.4 (RING2)
- new net: D45.2 (A), SW45.2
- new net: D20.2 (A), SW20.2
- new net: D38.2 (A), SW38.2
- new net: D26.2 (A), SW26.2
- new net: D5.2 (A), SW5.2
- new net: D36.2 (A), SW36.2
- new net: D35.2 (A), SW35.2
- new net: D7.2 (A), SW7.2
- new net: U1.17 (26), U3.3 (RING1)
- new net: U1.18 (27), U3.2 (TIP)
- new net: U1.22 (GND), U3.1 (SLEEVE)
- new net: U1.23 (5V), U3.4 (RING2)
- new net: D23.2 (A), SW23.2
- new net: D1.2 (A), SW1.2
- new net: D41.2 (A), SW41.2
- new net: D44.2 (A), SW44.2
- new net: D14.2 (A), SW14.2
- new net: D46.2 (A), SW46.2
- new net: D29.2 (A), SW29.2
- new net: D24.2 (A), SW24.2
- new net: D6.2 (A), SW6.2
- new net: D43.2 (A), SW43.2
- new net: D9.2 (A), SW9.2
- new net: D19.2 (A), SW19.2
- new net: D22.2 (A), SW22.2
- new net: D2.2 (A), SW2.2
- new net: D39.2 (A), SW39.2
- new net: D12.2 (A), SW12.2
- new net: D13.2 (A), SW13.2
- new net: D31.2 (A), SW31.2
- new net: D15.2 (A), SW15.2
- new net: D10.2 (A), SW10.2
- new net: D17.2 (A), SW17.2
- new net: D37.2 (A), SW37.2
- new net: D48.2 (A), SW48.2
- new net: D16.2 (A), SW16.2
- new net: D3.2 (A), SW3.2
- new net: D30.2 (A), SW30.2
- new net: D42.2 (A), SW42.2
- new net: D33.2 (A), SW33.2
- new net: D32.2 (A), SW32.2
- new net: D28.2 (A), SW28.2
- new net: D11.2 (A), SW11.2
- new net: D18.2 (A), SW18.2
- new net: D40.2 (A), SW40.2
- new net: D47.2 (A), SW47.2
- new net: D8.2 (A), SW8.2
- new net Lcol1: SW37.1, SW38.1, SW39.1, SW40.1, SW41.1, SW42.1, U2.6 (5)
- new net Lcol2: D26.1 (K), D32.1 (K), D38.1 (K), D44.1 (K), U2.9 (8)
- new net Lcol3: D28.1 (K), D34.1 (K), D40.1 (K), D46.1 (K), SW31.1, SW32.1, SW33.1, SW34.1, SW35.1, SW36.1
- new net Lcol4: D25.1 (K), D30.1 (K), D31.1 (K), D36.1 (K), D37.1 (K), D42.1 (K), D43.1 (K), D48.1 (K)
- new net Lrow1: D27.1 (K), D33.1 (K), D39.1 (K), D45.1 (K), U2.5 (4)
- new net Lrow2: SW43.1, SW44.1, SW45.1, SW46.1, SW47.1, SW48.1, U2.7 (6)
- new net Lrow3: U2.10 (9), U2.3 (2)
- new net Lrow4: U2.1 (0), U2.4 (3)
- new net Lrow5: SW25.1, SW26.1, SW27.1, SW28.1, SW29.1, SW30.1, U2.8 (7)
- new net Lrow6: D29.1 (K), D35.1 (K), D41.1 (K), D47.1 (K), U2.2 (1)
- new net RcoR1: SW13.1, SW14.1, SW15.1, SW16.1, SW17.1, SW18.1, U1.6 (5)
- new net RcoR2: D14.1 (K), D2.1 (K), D20.1 (K), D8.1 (K), U1.9 (8)
- new net RcoR3: D10.1 (K), D16.1 (K), D22.1 (K), D4.1 (K), SW10.1, SW11.1, SW12.1, SW7.1, SW8.1, SW9.1
- new net RcoR4: D1.1 (K), D12.1 (K), D13.1 (K), D18.1 (K), D19.1 (K), D24.1 (K), D6.1 (K), D7.1 (K)
- new net Rrow1: D15.1 (K), D21.1 (K), D3.1 (K), D9.1 (K), U1.5 (4)
- new net Rrow2: SW19.1, SW20.1, SW21.1, SW22.1, SW23.1, SW24.1, U1.7 (6)
- new net Rrow3: U1.10 (9), U1.3 (2)
- new net Rrow4: U1.1 (0), U1.4 (3)
- new net Rrow5: SW1.1, SW2.1, SW3.1, SW4.1, SW5.1, SW6.1, U1.8 (7)
- new net Rrow6: D11.1 (K), D17.1 (K), D23.1 (K), D5.1 (K), U1.2 (1)

Commit message: things
Parts:
- removed D1, D10, D11, D12, D13, D14, D15, D16, D17, D18, D19, D2, D20, D21, D22, D23, D24, D25, D26, D27, D28, D29, D3, D30, D31, D32, D33, D34, D35, D36, D37, D38, D39, D4, D40, D41, D42, D43, D44, D45, D46, D47, D48, D5, D6, D7, D8, D9: 1N4148WT, Diode_SMD:D_SOD-523, symbol Diode:1N4148WT
- removed SW1, SW10, SW11, SW12, SW13, SW14, SW15, SW16, SW17, SW18, SW19, SW2, SW20, SW21, SW22, SW23, SW24, SW25, SW26, SW27, SW28, SW29, SW3, SW30, SW31, SW32, SW33, SW34, SW35, SW36, SW37, SW38, SW39, SW4, SW40, SW41, SW42, SW43, SW44, SW45, SW46, SW47, SW48, SW5, SW6, SW7, SW8, SW9: Switch, ScottoKeebs_MX:MX_PCB_1.00u, symbol ScottoKeebs:Placeholder_Switch
- removed U1, U2: RP2040_Zero, ScottoKeebs_MCU:RP2040_Zero, symbol ScottoKeebs:MCU_RP2040_Zero
- removed U3, U4: TRRS, ScottoKeebs_Components:TRRS_PJ-320A, symbol ScottoKeebs:Placeholder_TRRS
- added LController1, RController1: ~, ScottoKeebs_MCU:Adafruit_KB2040, symbol ScottoKeebs:MCU_Adafruit_KB2040
- added LeftD1, LeftD10, LeftD11, LeftD12, LeftD13, LeftD14, LeftD15, LeftD16, LeftD17, LeftD18, LeftD19, LeftD2, LeftD3, LeftD4, LeftD5, LeftD6, LeftD7, LeftD8, LeftD9, RightD1, RightD10, RightD11, RightD12, RightD13, RightD14, RightD15, RightD16, RightD17, RightD18, RightD19, RightD2, RightD3, RightD4, RightD5, RightD6, RightD7, RightD8, RightD9: Diode, Diode_THT:D_DO-35_SOD27_P7.62mm_Horizontal, symbol ScottoKeebs:Placeholder_Diode
- added LeftSW1, LeftSW10, LeftSW11, LeftSW12, LeftSW13, LeftSW14, LeftSW15, LeftSW16, LeftSW17, LeftSW18, LeftSW19, LeftSW2, LeftSW3, LeftSW4, LeftSW5, LeftSW6, LeftSW7, LeftSW8, LeftSW9, RightSW1, RightSW10, RightSW11, RightSW12, RightSW13, RightSW14, RightSW15, RightSW16, RightSW17, RightSW18, RightSW19, RightSW2, RightSW3, RightSW4, RightSW5, RightSW6, RightSW7, RightSW8, RightSW9: Switch, ScottoKeebs_MX:MX_PCB_1.00u, symbol ScottoKeebs:Placeholder_Switch
Connections:
- new net: LeftD18.2 (A), LeftSW18.2
- new net: RightD3.2 (A), RightSW3.2
- new net: LeftD5.2 (A), LeftSW5.2
- new net: RightD11.2 (A), RightSW11.2
- new net: RightD14.2 (A), RightSW14.2
- new net: LeftD1.2 (A), LeftSW1.2
- new net: RightD16.2 (A), RightSW16.2
- new net: RightD2.2 (A), RightSW2.2
- new net: RightD13.2 (A), RightSW13.2
- new net: RightD1.2 (A), RightSW1.2
- new net: LeftD14.2 (A), LeftSW14.2
- new net: LeftD17.2 (A), LeftSW17.2
- new net: LeftD2.2 (A), LeftSW2.2
- new net: RightD10.2 (A), RightSW10.2
- new net: LeftD4.2 (A), LeftSW4.2
- new net: RightD4.2 (A), RightSW4.2
- new net: LeftD3.2 (A), LeftSW3.2
- new net: RightD5.2 (A), RightSW5.2
- new net: RightD18.2 (A), RightSW18.2
- new net: RightD15.2 (A), RightSW15.2
- new net: LeftD12.2 (A), LeftSW12.2
- new net: LeftD16.2 (A), LeftSW16.2
- new net: RightD9.2 (A), RightSW9.2
- new net: LeftD8.2 (A), LeftSW8.2
- new net: RightD6.2 (A), RightSW6.2
- new net: RightD12.2 (A), RightSW12.2
- new net: RightD7.2 (A), RightSW7.2
- new net: LeftD15.2 (A), LeftSW15.2
- new net: LeftD9.2 (A), LeftSW9.2
- new net: LeftD13.2 (A), LeftSW13.2
- new net: RightD17.2 (A), RightSW17.2
- new net: RightD8.2 (A), RightSW8.2
- new net: LeftD7.2 (A), LeftSW7.2
- new net: LeftD10.2 (A), LeftSW10.2
- new net: RightD19.2 (A), RightSW19.2
- new net: LeftD6.2 (A), LeftSW6.2
- new net: LeftD11.2 (A), LeftSW11.2
- new net: LeftD19.2 (A), LeftSW19.2
- new net LeftCol1: LController1.10 (6/PD7), LeftSW1.1, LeftSW2.1, LeftSW3.1, LeftSW4.1
- new net LeftCol2: LController1.11 (7/PE6), LeftSW5.1, LeftSW6.1, LeftSW7.1, LeftSW8.1
- new net LeftCol3: LController1.12 (8/PB4), LeftSW10.1, LeftSW11.1, LeftSW12.1, LeftSW9.1
- new net LeftCol4: LController1.13 (9/PB5), LeftSW13.1, LeftSW14.1, LeftSW15.1, LeftSW16.1
- new net LeftCol5: LController1.23 (15/PB1), LeftSW17.1, LeftSW18.1, LeftSW19.1
- new net LeftCol6: LController1.24 (14/PB3)
- new net LeftRow1: LController1.6 (2/PD1), LeftD1.1 (K), LeftD13.1 (K), LeftD5.1 (K), LeftD9.1 (K)
- new net LeftRow2: LController1.7 (3/PD0), LeftD10.1 (K), LeftD14.1 (K), LeftD17.1 (K), LeftD2.1 (K), LeftD6.1 (K)
- new net LeftRow3: LController1.8 (4/PD4), LeftD11.1 (K), LeftD15.1 (K), LeftD18.1 (K), LeftD3.1 (K), LeftD7.1 (K)
- new net LeftRow4: LController1.9 (5/PC6), LeftD12.1 (K), LeftD16.1 (K), LeftD19.1 (K), LeftD4.1 (K), LeftD8.1 (K)
- new net RightCol1: RController1.10 (6/PD7), RightSW16.1, RightSW17.1, RightSW18.1, RightSW19.1
- new net RightCol2: RController1.11 (7/PE6), RightSW12.1, RightSW13.1, RightSW14.1, RightSW15.1
- new net RightCol3: RController1.12 (8/PB4), RightSW10.1, RightSW11.1, RightSW8.1, RightSW9.1
- new net RightCol4: RController1.13 (9/PB5), RightSW4.1, RightSW5.1, RightSW6.1, RightSW7.1
- new net RightCol5: RController1.23 (15/PB1), RightSW1.1, RightSW2.1, RightSW3.1
- new net RightCol6: RController1.24 (14/PB3)
- new net RightRow1: RController1.6 (2/PD1), RightD12.1 (K), RightD16.1 (K), RightD4.1 (K), RightD8.1 (K)
- new net RightRow2: RController1.7 (3/PD0), RightD1.1 (K), RightD13.1 (K), RightD17.1 (K), RightD5.1 (K), RightD9.1 (K)
- new net RightRow3: RController1.8 (4/PD4), RightD10.1 (K), RightD14.1 (K), RightD18.1 (K), RightD2.1 (K), RightD6.1 (K)
- new net RightRow4: RController1.9 (5/PC6), RightD11.1 (K), RightD15.1 (K), RightD19.1 (K), RightD3.1 (K), RightD7.1 (K)
